File: esp32_wled_controller.kicad_pcb (KiCad board)
At the start: 4 copper layers, 95 x 95 mm, 83 parts, among them J1 USB_C_Receptacle_USB2.0_16P, J2 Screw_Terminal_01x03, J3 Screw_Terminal_01x03, J4 Screw_Terminal_01x03, J5 Screw_Terminal_01x03, J6 Screw_Terminal_01x02, J7 Screw_Terminal_01x02, K1 SRD-05VDC-SL-C, K2 SRD-05VDC-SL-C, K3 SRD-05VDC-SL-C, K4 SRD-05VDC-SL-C, Q1 SS8050, Q2 SS8050, Q3 SS8050, Q4 SS8050, Q5 SS8050, Q6 SS8050, SW1 SW_SPST, SW2 SW_SPST, U2 AMS1117-3.3, U3 CP2104, U4 EL817, U5 EL817, U6 EL817, U7 EL817, U8 ESP32-S2-WROOM-1-N4(4MB), U9 SN74AHCT125PWR

Commit message: inital rev 1.3 pcb design
Parts:
- removed 3.3V-PWR1: RED_LED, LED_SMD:LED_0805_2012Metric_Pad1.15x1.40mm_HandSolder
- removed 3V3, GND1, RX1, TX1: TestPoint, TestPoint:TestPoint_Pad_D1.5mm
- removed C10, C13: 22u, Capacitor_SMD:C_0805_2012Metric_Pad1.18x1.45mm_HandSolder
- removed C11, C12: 100nF, Capacitor_SMD:C_0402_1005Metric_Pad0.74x0.62mm_HandSolder
- removed G***1: LOGO, lib:wled-logo
- removed J1: USB_C_Receptacle_USB2.0_16P, Connector_USB:USB_C_Receptacle_G-Switch_GT-USB-7010ASV
- removed Q1, Q2: SS8050, Package_TO_SOT_SMD:SOT-23
- removed R10, R11: 22R, Resistor_SMD:R_0402_1005Metric_Pad0.72x0.64mm_HandSolder
- removed R5: 5K1, Resistor_SMD:R_0402_1005Metric_Pad0.72x0.64mm_HandSolder
- removed R9: 10K, Resistor_SMD:R_0402_1005Metric_Pad0.72x0.64mm_HandSolder
- removed REF**1: OSHW-Logo_11.4x12mm_SilkScreen, Symbol:OSHW-Logo_11.4x12mm_SilkScreen
- removed U3: CP2104, Package_DFN_QFN:QFN-24-1EP_4x4mm_P0.5mm_EP2.6x2.6mm
- removed U8: ESP32-S2-WROOM-1-N4(4MB), lib:WIFI-SMD_ESP32-S2-WROVER-I
- added AE2: ANT, RF_Antenna:Texas_SWRA117D_2.4GHz_Left, F.Cu at (87.9, 32.8)
- added C14: 10uF, Capacitor_SMD:C_0201_0603Metric_Pad0.64x0.40mm_HandSolder, F.Cu at (80.3, 44.8)
- added C15: 1uF, Capacitor_SMD:C_0402_1005Metric_Pad0.74x0.62mm_HandSolder, F.Cu at (79.0, 43.2)
- added C16: 1uF, Capacitor_SMD:C_0201_0603Metric_Pad0.64x0.40mm_HandSolder, F.Cu at (75.0, -1.61)
- added C17: 0.1uF, Capacitor_SMD:C_0402_1005Metric_Pad0.74x0.62mm_HandSolder, F.Cu at (79.7, 44.0)
- added C18: 2.2uF, Capacitor_SMD:C_0402_1005Metric_Pad0.74x0.62mm_HandSolder, F.Cu at (63.1, -1.11)
- added C19: 0.1uF, Capacitor_SMD:C_0402_1005Metric_Pad0.74x0.62mm_HandSolder, F.Cu at (82.7, 43.1)
- added C21: 10nF, Capacitor_SMD:C_0201_0603Metric_Pad0.64x0.40mm_HandSolder, F.Cu at (88.2, 44.1)
- added C22: 0.1uF, Capacitor_SMD:C_0402_1005Metric_Pad0.74x0.62mm_HandSolder, F.Cu at (81.8, 52.3)
- added C23: 1uF, Capacitor_SMD:C_0402_1005Metric_Pad0.74x0.62mm_HandSolder, F.Cu at (87.6, 43.2)
- added C28: 12pF, Capacitor_SMD:C_0201_0603Metric_Pad0.64x0.40mm_HandSolder, F.Cu at (76.4, -60.2)
- added C29: 12pF, Capacitor_SMD:C_0201_0603Metric_Pad0.64x0.40mm_HandSolder, F.Cu at (76.4, -58.5)
- added C30: 2.7pF, Capacitor_SMD:C_0201_0603Metric_Pad0.64x0.40mm_HandSolder, F.Cu at (84.9, 37.8)
- added C31: 0.1uF, Capacitor_SMD:C_0402_1005Metric_Pad0.74x0.62mm_HandSolder, F.Cu at (48.9, 39.4)
- added C32: 0.1uF, Capacitor_SMD:C_0402_1005Metric_Pad0.74x0.62mm_HandSolder, F.Cu at (90.2, 46.7)
- added C33: 0.1uF, Capacitor_SMD:C_0402_1005Metric_Pad0.74x0.62mm_HandSolder, F.Cu at (88.6, 53.5)
- added C34: 1uF, Capacitor_SMD:C_0402_1005Metric_Pad0.74x0.62mm_HandSolder, F.Cu at (87.7, 54.4)
- added C36: 3pF, Capacitor_SMD:C_0201_0603Metric_Pad0.64x0.40mm_HandSolder, F.Cu at (83.2, 37.8)
- added D4: PMEG6020AELR, Diode_SMD:Nexperia_CFP3_SOD-123W, F.Cu at (47.7, 41.3)
- added D5: CG0603MLU-24E, lib:R0603, F.Cu at (46.9, 43.4)
- added F1: 10A Fuse, Fuse:Fuseholder_Blade_Mini_Keystone_3568, F.Cu at (21.3, 97.4)
- added F2: 10A Fuse, Fuse:Fuseholder_Blade_Mini_Keystone_3568, F.Cu at (40.6, 97.4)
- added F3: 10A Fuse, Fuse:Fuseholder_Blade_Mini_Keystone_3568, F.Cu at (59.9, 97.4)
- added F4: 10A Fuse, Fuse:Fuseholder_Blade_Mini_Keystone_3568, F.Cu at (79.1, 97.4)
- added L1: 2nH, Inductor_SMD:L_0402_1005Metric, F.Cu at (82.0, 44.1)
- added L3: 6.8uH, lib:IND-SMD_L4.4-W4.2, F.Cu at (138.7, 49.0)
- added L4: 2.4nH, Inductor_SMD:L_0201_0603Metric, F.Cu at (87.4, 37.3)
- added PWR: RED_LED, LED_SMD:LED_0805_2012Metric_Pad1.15x1.40mm_HandSolder, F.Cu at (59.6, 35.2)
- added R24: 22, Resistor_SMD:R_0402_1005Metric, F.Cu at (72.8, -57.0)
- added R25: 5K1, Resistor_SMD:R_0402_1005Metric_Pad0.72x0.64mm_HandSolder, F.Cu at (55.5, 39.4)
- added R28: 5K1, Resistor_SMD:R_0402_1005Metric_Pad0.72x0.64mm_HandSolder, F.Cu at (50.8, 39.3)
- added SW3: SS12D10G4 071, lib:SW-TH_SHOU-HAN_SS12D10G4, F.Cu at (24.7, 48.9)
- added U1: ESP32-S3FH4R2, lib:QFN40P700X700X90-57N, F.Cu at (85.3, 48.8)
- added U10: USBLC6-2P6, Package_TO_SOT_SMD:SOT-666, F.Cu at (52.7, 40.3)
- added U11: TLV76733DRVx, Package_SON:WSON-6-1EP_2x2mm_P0.65mm_EP1x1.6mm_ThermalVias, F.Cu at (69.1, -0.76)
- added USB-C: USB_C_Receptacle_USB2.0_16P, Connector_USB:USB_C_Receptacle_G-Switch_GT-USB-7010ASV, F.Cu at (52.5, 32.2)
- added Y1: ECS-400-10-37B2-CKM-TR, Crystal:Crystal_SMD_2016-4Pin_2.0x1.6mm, F.Cu at (69.3, -58.0)
- C3, C9: value 22u -> 100nF; footprint Capacitor_SMD:C_0805_2012Metric_Pad1.18x1.45mm_HandSolder -> Capacitor_SMD:C_0402_1005Metric_Pad0.74x0.62mm_HandSolder
- C5: value 100nF -> 1uF
- C6: value 4u7 -> 1uF; footprint Capacitor_SMD:C_0805_2012Metric_Pad1.18x1.45mm_HandSolder -> Capacitor_SMD:C_0402_1005Metric_Pad0.74x0.62mm_HandSolder
- C7: value 22u -> 1uF; footprint Capacitor_SMD:C_0805_2012Metric_Pad1.18x1.45mm_HandSolder -> Capacitor_SMD:C_0402_1005Metric_Pad0.74x0.62mm_HandSolder
- C8: value 4u7 -> 47uF; footprint Capacitor_SMD:C_0805_2012Metric_Pad1.18x1.45mm_HandSolder -> Capacitor_SMD:C_0402_1005Metric_Pad0.74x0.62mm_HandSolder
- H6, H7, H8: value MountingHole_Pad -> MountingHole
- J6: value Screw_Terminal_01x02 -> VBUS_INPUT1
- J7: value Screw_Terminal_01x02 -> VBUS_INPUT2
- R1: value 10K -> 162k; footprint Resistor_SMD:R_0402_1005Metric_Pad0.72x0.64mm_HandSolder -> Resistor_SMD:R_0805_2012Metric_Pad1.20x1.40mm_HandSolder
- R2: value 10K -> 22.1k; footprint Resistor_SMD:R_0402_1005Metric_Pad0.72x0.64mm_HandSolder -> Resistor_SMD:R_0805_2012Metric_Pad1.20x1.40mm_HandSolder
- R4: value 5K1 -> 499
- U2: value AMS1117-3.3 -> LMR51430; footprint Package_TO_SOT_SMD:SOT-223-3_TabPin2 -> Package_TO_SOT_SMD:SOT-23-6
- moved H7 117.7 mm to (142.8, 103.3)
- moved R21 98.6 mm to (141.7, 72.8), turned to 0 degrees
- moved H6 87.2 mm to (15.5, 111.7)
- moved C1 83.6 mm to (94.8, -38.4), turned to 0 degrees
- moved SW1 82.9 mm to (104.8, -37.3)
- moved C2 74.8 mm to (94.8, -36.4), turned to 0 degrees
- moved R20 74.8 mm to (139.4, 73.8)
- moved R6 73.5 mm to (95.0, -31.4), turned to 0 degrees
- moved C8 73.0 mm to (137.1, 52.0)
- moved C4 70.8 mm to (137.5, 75.8), turned to 0 degrees
- moved C6 70.6 mm to (132.5, 45.4), turned to -90 degrees
- moved C5 70.5 mm to (130.1, 45.4), turned to -90 degrees
- moved SW2 69.9 mm to (104.8, -30.6), turned to 0 degrees
- moved C7 68.9 mm to (133.7, 45.4), turned to -90 degrees
- moved C9 68.1 mm to (132.6, 51.0), turned to 0 degrees
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Connections:
- net /EN renamed /CHIP_PU
- net /IO0 renamed /GPIO0
- C3 pad 1: +5V -> /9-24V
- C5 pad 1: +5V -> /9-24V
- C6 pad 1: +5V -> /9-24V
- C7 pad 1: +5V -> /9-24V
- C8 pad 1: Net-(U3-VPP) -> +5V
- C9 pad 1: +3.3V -> Net-(U2-CB)
- C9 pad 2: GND -> Net-(U2-SW)
- J2 pad 1: /STRIP1_5V -> /STRIP1_OUT
- J3 pad 1: /STRIP2_5V -> /STRIP2_OUT
- J4 pad 1: /STRIP3_5V -> unconnected-(J4-Pin_1-Pad1)
- J5 pad 1: /STRIP4_5V -> /STRIP4_OUT
- J6 pad 1: +5V -> /VBUS
- J7 pad 1: +5V -> /VBUS
- K1 pad NO: /STRIP1_5V -> /STRIP1_OUT_UF
- K2 pad NO: /STRIP2_5V -> /STRIP2_OUT_UF
- K3 pad NO: /STRIP3_5V -> /STRIP3_OUT_UF
- K4 pad NO: /STRIP4_5V -> /STRIP4_OUT_UF
- R1 pad 1: /RTS -> +5V
- R1 pad 2: Net-(Q1-B) -> Net-(U2-FB)
- R2 pad 1: /DTR -> Net-(U2-FB)
- R2 pad 2: Net-(Q2-B) -> GND
- R4 pad 2: GND -> Net-(U1-GPIO43/U0TXD)
- U2 pad 2: +3.3V -> Net-(U2-SW)
- U2 pad 3: +5V -> /9-24V
Routing:
- net +3.3V: track 87.8 -> 0.00 mm, vias 6 -> 0
- net GND: track 116.0 -> 36.9 mm, vias 17 -> 8
- net /RELAY1: track 78.0 -> 2.12 mm, vias 3 -> 1
- net /STRIP2: track 70.4 -> 0.00 mm, vias 2 -> 0
- net /STRIP1: track 65.7 -> 0.00 mm, vias 2 -> 0
- net /RELAY2: track 65.1 -> 2.12 mm, vias 3 -> 1
- net /CHIP_PU: track 60.8 -> 0.00 mm, vias 2 -> 0
- net /STRIP3: track 58.6 -> 0.00 mm
- net /STRIP4: track 57.6 -> 0.00 mm
- net /RELAY4: track 54.4 -> 2.12 mm, vias 3 -> 1
- net /RX: track 51.4 -> 0.00 mm, vias 2 -> 0
- net /TX: track 44.4 -> 0.00 mm, vias 2 -> 0
- net /RELAY3: track 41.0 -> 2.12 mm, vias 3 -> 1
- net Net-(U9-4Y): track 34.7 -> 0.00 mm
- net Net-(U9-1Y): track 30.9 -> 0.00 mm
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- removed copper zone on In2.Cu, net +5V
- removed copper zone on In1.Cu, net GND
Other:
- board size 95 x 95 mm -> 85 x 85 mm
- board text added: "VCC DATA GND"
- board text removed: "+5V DATA GND"
- board text removed: "3.3V"
- board text removed: "BOOT"
- board text removed: "ESP32-WLED-4ch-controller V1.2"
- board text removed: "GND"
- board text removed: "GND 5V"
- board text removed: "IO19"
- board text removed: "IO20"
- board text removed: "IO21"
- board text removed: "IO26"
- board text removed: "JLCJLCJLCJLC"
- board text removed: "KEEP-OUT ZONE"
- board text removed: "MADE WITH BY JACK0217"
- board text removed: "PWR"
- board text removed: "RE1"
- board text removed: "RE2"
- board text removed: "RE3"
- board text removed: "RESET"
- board text removed: "RX"
- board text removed: "TX"
- board text removed: "website: jack0217.dev github: @fellettigiacomo license: CERN-OHL-S"
- board text removed: "❤️"
