File: esp32_wled_controller.kicad_sch (KiCad schematic)
At the start: 82 parts, among them J1 USB_C_Receptacle_USB2.0_16P, J2 Screw_Terminal_01x03, J3 Screw_Terminal_01x03, J4 Screw_Terminal_01x03, J5 Screw_Terminal_01x03, J6 Screw_Terminal_01x02, J7 Screw_Terminal_01x02, K1 SRD-05VDC-SL-C, K2 SRD-05VDC-SL-C, K3 SRD-05VDC-SL-C, K4 SRD-05VDC-SL-C, Q1 SS8050, Q2 SS8050, Q3 BC547A, Q4 BC547A, Q5 BC547A, Q6 BC547A, U1 USBLC6-2P6, U2 AMS1117-3.3, U3 CP2104, U4 ESP32-SOLO1, U5 PC817, U6 PC817, U7 PC817, U8 PC817, U9 SN74AHCT125PWR

Commit message: board revision 1.1
Parts:
- removed C12: 100nF, Capacitor_SMD:C_0402_1005Metric_Pad0.74x0.62mm_HandSolder, symbol Device:C_Small
- removed H1, H2, H3, H4: MountingHole, MountingHole:MountingHole_2.7mm_M2.5_DIN965_Pad, symbol Mechanical:MountingHole
- removed R12: 1K, Resistor_SMD:R_0402_1005Metric_Pad0.72x0.64mm_HandSolder, symbol Device:R_Small
- removed RX1, TX1: TestPoint, TestPoint:TestPoint_Pad_D1.0mm, symbol Connector:TestPoint
- removed U4: ESP32-SOLO1, lib:ESP32SOLO1, symbol RF_Module:ESP32-WROOM-32U
- added GND2, RX2, TX2: TestPoint, TestPoint:TestPoint_Pad_D1.0mm, symbol Connector:TestPoint
- added H5, H6, H7, H8: MountingHole_Pad, MountingHole:MountingHole_2.5mm_Pad, symbol Mechanical:MountingHole_Pad
- added U10: ESP32-S2-WROOM, lib:XCVR_ESP32-S2-WROOM, symbol ESP32-S2-WROOM:ESP32-S2-WROOM
Connections:
- net +3.3V: now also U10.2 (3V3)
- net EN: now also U10.41 (EN)
- net GND: now also GND2.1, H5.1, H6.1, H7.1, H8.1, U10.1 (GND), U10.26 (GND__1), U10.42 (GND__2), U10.43 (GND__3), U10.44 (GND__4), U10.45 (GND__5), U10.46 (GND__6), U10.47 (GND__7), U10.48 (GND__8), U10.49 (GND__9), U10.50 (GND__10), U10.51 (GND__11)
- net IO0: now also U10.3 (IO0)
- net IO17_RELAYS: now also U10.20 (IO17)
- net RX: now also RX2.1, U10.38 (RXD0)
- net STRIP1: now also U10.23 (IO20)
- net STRIP2: now also U10.24 (IO21)
- net STRIP3: now also U10.22 (IO19)
- net STRIP4: now also U10.21 (IO18)
- net TX: now also TX2.1, U10.37 (TXD0)
- no-connect marks 0 -> 45
Other:
- note added: "07/05/2024"
- note added: "1.1"
- note added: "3.3V to 5V"
- note added: "BJT"
- note added: "BUTTONS"
- note added: "ESP32"
- note added: "ESP32 WLED CONTROLLER"
- note added: "HEADERS AND HOLES"
- note added: "LEVEL SHIFTER"
- note added: "PWR LED"
- note added: "RELEAYS"
- note added: "USB TO SERIAL CONVERTER"
- moved on the sheet: 3.3V-PWR1, C1, C10, C11, C2, C3, C4, C5, C6, C7, C8, C9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

Commit message: board rev 1.2, cleanup
Parts:
- removed 3.3V1, GND2, RX2, TX2: TestPoint, TestPoint:TestPoint_Pad_D1.0mm, symbol Connector:TestPoint
- removed C14: 100nF, Capacitor_SMD:C_0402_1005Metric_Pad0.74x0.62mm_HandSolder, symbol Device:C_Small
- removed D5, D6, D7: 1N4007, Diode_SMD:D_MELF_Handsoldering, symbol local_lib:1N4007
- removed H5: MountingHole_Pad, MountingHole:MountingHole_2.5mm_Pad, symbol Mechanical:MountingHole_Pad
- removed Q3, Q4, Q5, Q6: BC547A, Package_TO_SOT_SMD:TSOT-23_HandSoldering, symbol local_lib:BC547A
- removed U10: ESP32-S2-WROOM, lib:XCVR_ESP32-S2-WROOM, symbol ESP32-S2-WROOM:ESP32-S2-WROOM
- removed U5, U6, U7, U8: PC817, Package_DIP:SMDIP-4_W7.62mm, symbol local_lib:PC817
- added 3V3, RX1, TX1: TestPoint, TestPoint:TestPoint_Pad_D1.5mm, symbol Connector:TestPoint
- added C12: 100nF, Capacitor_SMD:C_0402_1005Metric_Pad0.74x0.62mm_HandSolder, symbol Device:C_Small
- added D1, D2, D3: C7420350, Diode_SMD:D_MELF_Handsoldering, symbol local_lib:1N4007
- added JP1, JP2, JP3: SolderJumper_2_Bridged, Jumper:SolderJumper-2_P1.3mm_Open_TrianglePad1.0x1.5mm, symbol Jumper:SolderJumper_2_Bridged
- added Q3, Q4, Q5, Q6: SS8050, Package_TO_SOT_SMD:SOT-23, symbol Device:Q_NPN_BEC
- added U4, U5, U6, U7: EL817, Package_DIP:DIP-4_W7.62mm, symbol Isolator:EL817
- added U8: ESP32-S2-WROOM-1-N4(4MB), lib:WIFI-SMD_ESP32-S2-WROVER-I, symbol ESP32:ESP32-S2-WROOM-1-N4(4MB)
- C1, C11, C2, C4, C5: LCSC (none) -> C1525
- C10, C13, C3, C7, C9: LCSC (none) -> C45783
- C6, C8: LCSC (none) -> C1779
- D9: value 1N4007 -> C7420350; LCSC (none) -> C7420350
- GND1: footprint TestPoint:TestPoint_Pad_D1.0mm -> TestPoint:TestPoint_Pad_D1.5mm
- J1: LCSC (none) -> C2988369
- K1, K2, K3, K4: LCSC (none) -> C35449
- Q1, Q2: LCSC (none) -> C431710
- R1, R2, R9: LCSC (none) -> C25744
- R10, R11: LCSC (none) -> C25092
- R13, R14, R15, R16, R17, R18, R19, R3, R6, R7, R8: LCSC (none) -> C17513
- R20, R21, R22, R23: LCSC (none) -> C25076
- R4, R5: LCSC (none) -> C25905
- RELAY1, RELAY2, RELAY3, RELAY4: LCSC (none) -> C84256
- U1: LCSC (none) -> C2827693
- U2: LCSC (none) -> C6186
- U3: LCSC (none) -> C47742
- U9: LCSC (none) -> C36365
Connections:
- net +3.3V: now also 3V3.1, C12.1, U8.2 (3V3)
- net +5V: now also C4.2, U9.14 (VCC), D1.1 (K), D2.1 (K), D3.1 (K), U4.4, U5.4, U6.4, U7.4
- net EN: now also U8.41 (EN)
- net GND: now also C4.1, U9.1 (~{1OE}), U9.10 (~{3OE}), U9.13 (~{4OE}), U9.4 (~{2OE}), U9.7 (GND), C12.2, Q3.2 (E), Q4.2 (E), Q5.2 (E), Q6.2 (E), U8.1 (GND)
- net IO0: now also U8.3 (IO0)
- net RX: now also RX1.1, U8.38 (RXD0)
- net STRIP1: now also U8.24 (IO21)
- net STRIP2: now also U8.25 (IO26)
- net STRIP3: now also U8.23 (IO20)
- net STRIP4: now also U8.22 (IO19)
- net TX: now also TX1.1, U8.37 (TXD0)
- net at R8.1: now also U7.1
- net at RELAY1.2 (A): now also U7.2
- net at R15.1: now also U7.3
- net at K3.A2: now also D1.2 (A), Q5.3 (C)
- net at D9.2 (A), K4.A2: now also Q6.3 (C)
- net at R19.2: now also Q6.1 (B)
- net at K2.A2: now also D2.2 (A), Q4.3 (C)
- net at R19.1: now also U5.3
- net at R16.2: now also Q4.1 (B)
- net at K1.A2: now also D3.2 (A), Q3.3 (C)
- net at R15.2: now also Q3.1 (B)
- net at R13.1: now also U6.1
- net at RELAY4.2 (A): now also U5.2
- net at RELAY3.2 (A): now also U4.2
- net at RELAY2.2 (A): now also U6.2
- net at R17.2: now also Q5.1 (B)
- net at R14.1: now also U4.1
- net at R17.1: now also U4.3
- net at R18.1: now also U5.1
- net at R16.1: now also U6.3
- removed net IO17_RELAYS: RELAY1.1 (K), RELAY2.1 (K), RELAY3.1 (K), RELAY4.1 (K)
- new net RELAY1: JP3.2 (B), RELAY1.1 (K), U8.18 (IO15)
- new net RELAY2: JP2.2 (B), RELAY2.1 (K), U8.19 (IO16)
- new net RELAY3: JP1.2 (B), RELAY3.1 (K), U8.20 (IO17)
- new net RELAY4: JP1.1 (A), JP2.1 (A), JP3.1 (A), RELAY4.1 (K), U8.21 (IO18)
Other:
- note added: "1.2"
- note added: "24/05/2024"
- note added: "C106900"
- note added: "C431710"
- note added: "M7"
- note removed: "07/05/2024"
- note removed: "1.1"

Commit message: changed terminal block footprint
Parts:
- J2, J3, J4, J5: footprint TerminalBlock_Phoenix:TerminalBlock_Phoenix_MKDS-1,5-3-5.08_1x03_P5.08mm_Horizontal -> lib:CONN-TH_3P-P5.00_KF301-5.0-3P
- J6, J7: footprint TerminalBlock_Phoenix:TerminalBlock_Phoenix_MKDS-1,5-2-5.08_1x02_P5.08mm_Horizontal -> lib:CONN-TH_P5.00_KF301-5.0-2P
Changed lines of the file:
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@@
 			)
 		)
-		(property "Footprint" "TerminalBlock_Phoenix:TerminalBlock_Phoenix_MKDS-1,5-3-5.08_1x03_P5.08mm_Horizontal"
+		(property "Footprint" "lib:CONN-TH_3P-P5.00_KF301-5.0-3P"
 			(at 283.21 158.75 0)
 			(effects
@@
 			)
 		)
-		(property "Footprint" "TerminalBlock_Phoenix:TerminalBlock_Phoenix_MKDS-1,5-2-5.08_1x02_P5.08mm_Horizontal"
+		(property "Footprint" "lib:CONN-TH_P5.00_KF301-5.0-2P"
 			(at 331.47 142.24 0)
 			(effects
@@
 			)
 		)
-		(property "Footprint" "TerminalBlock_Phoenix:TerminalBlock_Phoenix_MKDS-1,5-3-5.08_1x03_P5.08mm_Horizontal"
+		(property "Footprint" "lib:CONN-TH_3P-P5.00_KF301-5.0-3P"
 			(at 283.21 140.97 0)
 			(effects
@@
 			)
 		)
-		(property "Footprint" "TerminalBlock_Phoenix:TerminalBlock_Phoenix_MKDS-1,5-3-5.08_1x03_P5.08mm_Horizontal"
+		(property "Footprint" "lib:CONN-TH_3P-P5.00_KF301-5.0-3P"
 			(at 283.21 123.19 0)
 			(effects
@@
 			)
 		)
-		(property "Footprint" "TerminalBlock_Phoenix:TerminalBlock_Phoenix_MKDS-1,5-3-5.08_1x03_P5.08mm_Horizontal"
+		(property "Footprint" "lib:CONN-TH_3P-P5.00_KF301-5.0-3P"
 			(at 283.21 176.53 0)
 			(effects
@@
 			)
 		)
-		(property "Footprint" "TerminalBlock_Phoenix:TerminalBlock_Phoenix_MKDS-1,5-2-5.08_1x02_P5.08mm_Horizontal"
+		(property "Footprint" "lib:CONN-TH_P5.00_KF301-5.0-2P"
 			(at 331.47 124.46 0)
 			(effects

Commit message: final 1.2 release
Parts:
- removed SW-BOOT1, SW-RESET1: SW_SPST, lib:TS-1187A-B-A-B, symbol Switch:SW_SPST
- removed U1: USBLC6-2P6, Package_TO_SOT_SMD:SOT-666, symbol Power_Protection:USBLC6-2P6
- added SW1, SW2: SW_SPST, Button_Switch_SMD:SW_Push_1P1T_XKB_TS-1187A, symbol Switch:SW_SPST
Connections:
- net EN: now also SW1.2 (B)
- net GND: now also U8.42 (GND), U8.43 (GND), SW1.1 (A), SW2.1 (A); no longer J1.S1 (SHIELD)
- net IO0: now also SW2.2 (B)
- net D-: now reaches J1.A7 (D-), J1.B7 (D-)
- net D-: now also U3.4 (D-)
- net D+: now reaches J1.A6 (D+), J1.B6 (D+)
- net D+: now also U3.3 (D+)
- no-connect marks 45 -> 44
Other:
- moved on the sheet: J1, R5

Commit message: fix optocoupler footprint, fix layout
Parts:
- U4, U5, U6, U7: footprint Package_DIP:DIP-4_W7.62mm -> lib:OPTO-SMD-4_L4.6-W6.5-P2.54-LS10.3-TL
Changed lines of the file:
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@@
 			)
 		)
-		(property "Footprint" "Package_DIP:DIP-4_W7.62mm"
+		(property "Footprint" "lib:OPTO-SMD-4_L4.6-W6.5-P2.54-LS10.3-TL"
 			(at 54.61 57.15 0)
 			(effects
@@
 			)
 		)
-		(property "Footprint" "Package_DIP:DIP-4_W7.62mm"
+		(property "Footprint" "lib:OPTO-SMD-4_L4.6-W6.5-P2.54-LS10.3-TL"
 			(at 54.61 198.12 0)
 			(effects
@@
 			)
 		)
-		(property "Footprint" "Package_DIP:DIP-4_W7.62mm"
+		(property "Footprint" "lib:OPTO-SMD-4_L4.6-W6.5-P2.54-LS10.3-TL"
 			(at 54.61 102.87 0)
 			(effects
@@
 			)
 		)
-		(property "Footprint" "Package_DIP:DIP-4_W7.62mm"
+		(property "Footprint" "lib:OPTO-SMD-4_L4.6-W6.5-P2.54-LS10.3-TL"
 			(at 54.61 148.59 0)
 			(effects

Commit message: add rev 1.3 schematic: esp32 chip, pcb chip antenna, boost converter
Parts:
- removed 3V3, GND1, RX1, TX1: TestPoint, TestPoint:TestPoint_Pad_D1.5mm, symbol Connector:TestPoint
- removed C10, C13: 22u, Capacitor_SMD:C_0805_2012Metric_Pad1.18x1.45mm_HandSolder, symbol Device:C_Small
- removed C11, C12: 100nF, Capacitor_SMD:C_0402_1005Metric_Pad0.74x0.62mm_HandSolder, symbol Device:C_Small
- removed J1: USB_C_Receptacle_USB2.0_16P, Connector_USB:USB_C_Receptacle_G-Switch_GT-USB-7010ASV, symbol Connector:USB_C_Receptacle_USB2.0_16P
- removed Q1, Q2: SS8050, Package_TO_SOT_SMD:SOT-23, symbol Device:Q_NPN_BEC
- removed R10, R11: 22R, Resistor_SMD:R_0402_1005Metric_Pad0.72x0.64mm_HandSolder, symbol Device:R_Small
- removed R4, R5: 5K1, Resistor_SMD:R_0402_1005Metric_Pad0.72x0.64mm_HandSolder, symbol Device:R_Small
- removed R9: 10K, Resistor_SMD:R_0402_1005Metric_Pad0.72x0.64mm_HandSolder, symbol Device:R_Small
- removed U2: AMS1117-3.3, Package_TO_SOT_SMD:SOT-223-3_TabPin2, symbol Regulator_Linear:LM1117MP-3.3
- removed U3: CP2104, Package_DFN_QFN:QFN-24-1EP_4x4mm_P0.5mm_EP2.6x2.6mm, symbol Interface_USB:CP2104
- removed U8: ESP32-S2-WROOM-1-N4(4MB), lib:WIFI-SMD_ESP32-S2-WROVER-I, symbol ESP32:ESP32-S2-WROOM-1-N4(4MB)
- added ANT1: 2450AT18D0100E, lib:ANT-SMD_4P-L3.2-W1.6, symbol 2450AT18D0100E:2450AT18D0100E
- added C14: 10uF, Capacitor_SMD:C_0201_0603Metric_Pad0.64x0.40mm_HandSolder, symbol Device:C
- added C15, C23, C34: 1uF, Capacitor_SMD:C_0402_1005Metric_Pad0.74x0.62mm_HandSolder, symbol Device:C
- added C16: 1uF, Capacitor_SMD:C_0201_0603Metric_Pad0.64x0.40mm_HandSolder, symbol Device:C
- added C17, C19, C22, C31, C32, C33: 0.1uF, Capacitor_SMD:C_0402_1005Metric_Pad0.74x0.62mm_HandSolder, symbol Device:C
- added C18: 2.2uF, Capacitor_SMD:C_0402_1005Metric_Pad0.74x0.62mm_HandSolder, symbol Device:C
- added C21: 10nF, Capacitor_SMD:C_0201_0603Metric_Pad0.64x0.40mm_HandSolder, symbol Device:C
- added C24, C25: NC, Capacitor_SMD:C_0201_0603Metric_Pad0.64x0.40mm_HandSolder, symbol Device:C
- added C26: 2.4pF, Capacitor_SMD:C_0201_0603Metric_Pad0.64x0.40mm_HandSolder, symbol Device:C
- added C27: 2.7pF, Capacitor_SMD:C_0201_0603Metric_Pad0.64x0.40mm_HandSolder, symbol Device:C
- added C28, C29: 12pF, Capacitor_SMD:C_0201_0603Metric_Pad0.64x0.40mm_HandSolder, symbol Device:C
- added D4: PMEG6020AELR, Diode_SMD:Nexperia_CFP3_SOD-123W, symbol Diode:PMEG6020AELR
- added D5: CG0603MLU-24E, lib:R0603, symbol CG0603MLU-24E:CG0603MLU-24E
- added J9: USB_C_Receptacle_USB2.0_16P, Connector_USB:USB_C_Receptacle_G-Switch_GT-USB-7010ASV, symbol Connector:USB_C_Receptacle_USB2.0_16P
- added L1: 2nH, Inductor_SMD:L_0402_1005Metric, symbol Device:L
- added L2: 2.4nH, Inductor_SMD:L_0201_0603Metric, symbol Device:L
- added L3: 6.8uH, lib:IND-SMD_L4.4-W4.2, symbol Device:L
- added R12: 0, Resistor_SMD:R_0201_0603Metric, symbol Device:R
- added R24: 22, Resistor_SMD:R_0402_1005Metric, symbol Device:R
- added R25, R28: 5K1, Resistor_SMD:R_0402_1005Metric_Pad0.72x0.64mm_HandSolder, symbol Device:R_Small
- added SW3: SS12D10G4 071, lib:SW-TH_SHOU-HAN_SS12D10G4, symbol easyeda2kicad:SS12D10G4071
- added U1: ESP32-S3FH4R2, lib:QFN40P700X700X90-57N, symbol ESP32-S3FH4R2:ESP32-S3FH4R2
- added U10: USBLC6-2P6, Package_TO_SOT_SMD:SOT-666, symbol Power_Protection:USBLC6-2P6
- added U11: TLV76733DRVx, Package_SON:WSON-6-1EP_2x2mm_P0.65mm_EP1x1.6mm_ThermalVias, symbol Regulator_Linear:TLV76733DRVx
- added U2: LMR51430, Package_TO_SOT_SMD:SOT-23-6, symbol Regulator_Switching:LMR51430
- added Y1: ECS-400-10-37B2-CKM-TR, Crystal:Crystal_SMD_2016-4Pin_2.0x1.6mm, symbol Device:Crystal_GND24_Small
- C3, C9: value 22u -> 100nF; footprint Capacitor_SMD:C_0805_2012Metric_Pad1.18x1.45mm_HandSolder -> Capacitor_SMD:C_0402_1005Metric_Pad0.74x0.62mm_HandSolder; LCSC C45783 -> (none)
- C5: value 100nF -> 1uF; LCSC C1525 -> (none)
- C6: value 4u7 -> 1uF; footprint Capacitor_SMD:C_0805_2012Metric_Pad1.18x1.45mm_HandSolder -> Capacitor_SMD:C_0402_1005Metric_Pad0.74x0.62mm_HandSolder; LCSC C1779 -> (none)
- C7: value 22u -> 1uF; footprint Capacitor_SMD:C_0805_2012Metric_Pad1.18x1.45mm_HandSolder -> Capacitor_SMD:C_0402_1005Metric_Pad0.74x0.62mm_HandSolder; LCSC C45783 -> (none)
- C8: value 4u7 -> 47uF; footprint Capacitor_SMD:C_0805_2012Metric_Pad1.18x1.45mm_HandSolder -> Capacitor_SMD:C_0402_1005Metric_Pad0.74x0.62mm_HandSolder; LCSC C1779 -> (none); now fitted; now in the parts list
- R1: value 10K -> 162k; footprint Resistor_SMD:R_0402_1005Metric_Pad0.72x0.64mm_HandSolder -> Resistor_SMD:R_0805_2012Metric_Pad1.20x1.40mm_HandSolder; LCSC C25744 -> (none)
- R2: value 10K -> 22.1k; footprint Resistor_SMD:R_0402_1005Metric_Pad0.72x0.64mm_HandSolder -> Resistor_SMD:R_0805_2012Metric_Pad1.20x1.40mm_HandSolder; LCSC C25744 -> (none)
Connections:
- net DTR is gone; now on an unnamed net: R2.1
- net RTS is gone; now on net +5V: R1.1
- net +3.3V: no longer C9.1
- net +5V: now also C8.1, C16.1, D4.1 (K), D5.1 (K), L3.2, SW3.3, U11.4 (EN), U11.6 (IN); no longer C3.1, C5.1, C6.1, C7.1, J6.1 (Pin_1), J7.1 (Pin_1)
- net D+: now also U1.26 (GPIO20), U10.4 (I/O2)
- net D-: now also U1.25 (GPIO19), U10.6 (I/O1)
- net GND: now also R2.2, ANT1.2 (GND_1), ANT1.3 (GND_2), ANT1.4 (GND/FEED), C14.2, C15.2, C16.2, C17.2, C18.2, C19.2, C21.2, C22.2, C23.2, C24.2, C25.2, C26.2, C27.2, C28.2, C29.2, C31.2, C32.2, C33.2, C34.2, D5.2 (A), R25.2, R28.2, U1.57 (GND), U10.2 (GND), U11.3 (GND), U11.5 (GND), U11.7 (PAD), U2.1 (GND), Y1.2, Y1.4; no longer C9.2
- net RELAY1: now also U1.10 (GPIO5)
- net RELAY2: now also U1.11 (GPIO6)
- net RELAY3: now also U1.12 (GPIO7)
- net RELAY4: now also U1.13 (GPIO8)
- net STRIP1: now also U1.6 (GPIO1)
- net STRIP2: now also U1.7 (GPIO2)
- net STRIP3: now also U1.8 (GPIO3)
- net STRIP4: now also U1.9 (GPIO4)
- net at R1.2: now also U2.4 (FB)
- net EN renamed CHIP_PU
- net CHIP_PU: now also U1.4 (CHIP_PU)
- net IO0 renamed GPIO0
- net GPIO0: now also U1.5 (GPIO0)
- net STRIP1_5V renamed STRIP1_OUT
- net STRIP2_5V renamed STRIP2_OUT
- net STRIP3_5V renamed STRIP3_OUT
- net STRIP4_5V renamed STRIP4_OUT
- new net: C9.1, U2.6 (CB)
- new net: C9.2, L3.1, U2.2 (SW)
- new net: C25.1, C26.1, L2.2, R12.1
- new net: C28.1, R24.2, Y1.1
- new net: ANT1.1 (FEED/GND), C24.1, R12.2
- new net: J9.A7 (D-), J9.B7 (D-), U10.1 (I/O1)
- new net: J9.A6 (D+), J9.B6 (D+), U10.3 (I/O2)
- new net: C31.1, D4.2 (A), J9.A4 (VBUS), J9.A9 (VBUS), J9.B4 (VBUS), J9.B9 (VBUS), U10.5 (VBUS)
- new net: J9.A1 (GND), J9.A12 (GND), J9.B1 (GND), J9.B12 (GND)
- new net: J9.A5 (CC1), R25.1
- new net: J9.B5 (CC2), R28.1
- new net +3V3: C14.1, C15.1, C17.1, C18.1, C21.1, C22.1, C23.1, C32.1, C33.1, C34.1, L1.1, U1.20 (VDD3P3_RTC), U1.29 (VDD_SPI), U1.46 (VDD3P3_CPU), U1.55 (VDDA), U1.56 (VDDA__1), U11.1 (OUT), U11.2 (SNS)
- new net 9-24V: C3.1, C5.1, C6.1, C7.1, SW3.1, U2.3 (VIN), U2.5 (EN)
- new net LNA_IN: C27.1, L2.1, U1.1 (LNA_IN)
- new net VBUS: J6.1 (Pin_1), J7.1 (Pin_1), SW3.2
- new net VDD3P3: C19.1, L1.2, U1.2 (VDD3P3), U1.3 (VDD3P3__1)
- new net XTAL_N: C29.1, U1.53 (XTAL_N), Y1.3
- new net XTAL_P: R24.1, U1.54 (XTAL_P)
- no-connect marks 44 -> 41
Other:
- note added: "40MHZ CLOCK"
- note added: "BUCK CONVERTER (9-24V -> 5V)"
- note added: "ESP32-S3 MCU"
- note added: "LDO (5V -> 3.3V)"
- note added: "MCU POWER"
- note added: "PCB ANTENNA"
- note added: "USB-C INTERFACE / ESD PROTECTION"
- note removed: "1.2"
- note removed: "24/05/2024"
- note removed: "3.3V to 5V"
- note removed: "BJT"
- note removed: "C431710"
- note removed: "ESP32"
- note removed: "USB TO SERIAL CONVERTER"
- company: (none) -> jack0217.dev
- title: (none) -> ESP32-4CH-WLED-CONTROLLER
- moved on the sheet: 3.3V-PWR1, C1, C2, C4, H6, H7, H8, J2, J3, J4, J5, J6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
